File: kicad/ESP3D SHIELD/ESP3D SHIELD.kicad_pcb (KiCad board)
At the start: 2 copper layers, 38.7 x 19.1 mm, 12 parts, among them Q1 BSS138, Q2 BSS138, SW1 RESET, SW2 PROGRAM, SW3 RESET_CONFIG, U1 LM1117-3.3, U2 ESP-12E

Commit message: connector is now IDC , bigger board
Parts:
- added REF***: OSHW-Logo2_7.3x6mm_SilkScreen, Symbols:OSHW-Logo2_7.3x6mm_SilkScreen, F.Cu at (210.6, 124.6)
- AUX1: footprint Socket_Strips:Socket_Strip_Straight_2x04_Pitch2.54mm -> Connectors:IDC_Header_Straight_8pins; moved to F.Cu
- moved AUX1 8.26 mm to (227.3, 122.6), turned to 90 degrees
Connections:
- AUX1 pad 1: /HL1 -> (no net)
- AUX1 pad 2: (no net) -> +5V
- AUX1 pad 3: /HL2 -> (no net)
- AUX1 pad 4: (no net) -> GND
- AUX1 pad 5: GND -> (no net)
- AUX1 pad 6: (no net) -> /HL2
- AUX1 pad 7: +5V -> (no net)
- AUX1 pad 8: (no net) -> /HL1
Routing:
- net GND: track 77.5 -> 79.4 mm
- net /HL2: track 29.7 -> 30.8 mm
- net +5V: track 25.8 -> 26.9 mm
- net /HL1: track 25.1 -> 25.7 mm
Other:
- board size 38.7 x 19.1 mm -> 45.8 x 19.1 mm
- board text added: "ESP3D-SHIELD"
- board text added: "GPLv3"
- board text added: "PROG"
- board text added: "RESET"
- board text added: "Rx‹"
- board text added: "Tx›"
- board text removed: "AUX-1"
- board text removed: "ESP3D"
- board text removed: "PRG"
- board text removed: "RST"
- board text removed: "‹Tx"
- board text removed: "›Rx"
